File: spot_welder.sch (EAGLE design)
At the start: 38 parts, among them IC1 ATMEGA328PU, IC2 7805L, IC3 MOC3052M, T1 BT151-800R, T2 BT151-800R, Y1 16MHZ

Commit message: rerouted
Parts:
- removed TIME_SWITCH: Time switch, SparkFun-Connectors:M05LOCK
- added S5: Time switch, SparkFun-Connectors:M05NO_SILK
- C5, C6: device SparkFun-Passives:CAPPTH1 -> rcl:C-EU025-024X044
- JP5: device SparkFun-Connectors:M07LOCK -> SparkFun-Connectors:M07NO_SILK
Connections:
- net GND: now also JP5.1, S5.5; no longer JP5.7, TIME_SWITCH.1
- net N$18: now also S5.4; no longer TIME_SWITCH.5
- net N$23: now also S5.3; no longer TIME_SWITCH.4
- net N$24: now also S5.2; no longer TIME_SWITCH.3
- net N$25: now also S5.1; no longer TIME_SWITCH.2
- net VCC: now also JP5.7; no longer JP5.1
